Commit message: Working

File: src/my_robot/urdf/my_robot.xacro (robot description, xacro)
@@ -21,5 +21,5 @@
       <origin xyz="0 0 0" rpy=" 0 0 0"/>
       <geometry>
-        <box size=".4 .2 .1"/>
+        <box size=".4 .2 .05"/>
       </geometry>
     </collision>
@@ -27,29 +27,29 @@
       <origin xyz="0 0 0" rpy=" 0 0 0"/>
       <geometry>
-        <box size=".4 .2 .1"/>
+        <box size=".4 .2 .05"/>
       </geometry>
     </visual>
     <collision name='back_caster_collision'>
-      <origin xyz="-0.15 0 -0.05" rpy=" 0 0 0"/>
+      <origin xyz="-0.15 0 -0.03" rpy=" 0 0 0"/>
       <geometry>
-        <sphere radius="0.0499"/>
+        <sphere radius="0.0199"/>
       </geometry>
     </collision>
     <visual name='back_caster_visual'>
-      <origin xyz="-0.15 0 -0.05" rpy=" 0 0 0"/>
+      <origin xyz="-0.15 0 -0.03" rpy=" 0 0 0"/>
       <geometry>
-        <sphere radius="0.05"/>
+        <sphere radius="0.02"/>
       </geometry>
     </visual>
     <collision name='front_caster_collision'>
-      <origin xyz="0.15 0 -0.05" rpy=" 0 0 0"/>
+      <origin xyz="0.15 0 -0.03" rpy=" 0 0 0"/>
       <geometry>
-        <sphere radius="0.0499"/>
+        <sphere radius="0.0199"/>
       </geometry>
     </collision>
     <visual name='front_caster_visual'>
-      <origin xyz="0.15 0 -0.05" rpy=" 0 0 0"/>
+      <origin xyz="0.15 0 -0.03" rpy=" 0 0 0"/>
       <geometry>
-        <sphere radius="0.05"/>
+        <sphere radius="0.02"/>
       </geometry>
     </visual>
@@ -68,5 +68,5 @@
       <origin xyz="0 0 0" rpy="0 1.5707 1.5707"/>
     <geometry>
-      <cylinder radius="0.05" length="0.05"/>
+      <cylinder radius="0.05" length="0.02"/>
     </geometry>
     </collision>
@@ -74,5 +74,5 @@
       <origin xyz="0 0 0" rpy="0 1.5707 1.5707"/>
     <geometry>
-      <cylinder radius="0.05" length="0.05"/>
+      <cylinder radius="0.05" length="0.02"/>
     </geometry>
     </visual>
@@ -91,5 +91,5 @@
       <origin xyz="0 0 0" rpy="0 1.5707 1.5707"/>
     <geometry>
-      <cylinder radius="0.05" length="0.05"/>
+      <cylinder radius="0.05" length="0.02"/>
     </geometry>
     </collision>
@@ -97,10 +97,10 @@
       <origin xyz="0 0 0" rpy="0 1.5707 1.5707"/>
     <geometry>
-      <cylinder radius="0.05" length="0.05"/>
+      <cylinder radius="0.05" length="0.02"/>
     </geometry>
     </visual>
   </link>
   <joint type="continuous" name="left_wheel_hinge">
-    <origin xyz="0 0.15 0" rpy="0 0 0"/>
+    <origin xyz="0 0.112 0" rpy="0 0 0"/>
     <child link="left_wheel"/>
     <parent link="chassis"/>
@@ -110,5 +110,5 @@
   </joint>
   <joint type="continuous" name="right_wheel_hinge">
-    <origin xyz="0 -0.15 0" rpy="0 0 0"/>
+    <origin xyz="0 -0.112 0" rpy="0 0 0"/>
     <child link="right_wheel"/>
     <parent link="chassis"/>
@@ -121,5 +121,5 @@
       <origin xyz="0 0 0" rpy="0 0 0"/>
       <geometry>
-        <box size="0.05 0.05 0.05"/>
+        <box size="0.05 0.04 0.04"/>
       </geometry>
     </visual>
@@ -167,10 +167,10 @@
   <joint name="hokuyo_joint" type="fixed">
     <axis xyz="0 1 0"/>
-    <origin xyz="0.15 0 0.1" rpy="0 0 0"/>
+    <origin xyz="0.15 0 0.02" rpy="0 0 0"/>
     <parent link="chassis"/>
     <child link="hokuyo"/>
   </joint>
   <gazebo reference="chassis">
-    <material>Gazebo/Chrome</material>
+    <material>Gazebo/Blue</material>
   </gazebo>
   <gazebo reference="left_wheel">

Commit message: submit 2

File: src/my_robot/urdf/my_robot.xacro (robot description, xacro)
@@ -167,5 +167,5 @@
   <joint name="hokuyo_joint" type="fixed">
     <axis xyz="0 1 0"/>
-    <origin xyz="0.15 0 0.02" rpy="0 0 0"/>
+    <origin xyz="0.17 0 0.06" rpy="0 0 0"/>
     <parent link="chassis"/>
     <child link="hokuyo"/>

Commit message: Home Service Robot

File: src/my_robot/urdf/my_robot.xacro (robot description, xacro)
@@ -144,4 +144,30 @@
     <child link="camera"/>
   </joint>
+  <joint name="camera_optical_joint" type="fixed">
+    <origin xyz="0 0 0" rpy="-1.5707 0 -1.5707"/>
+    <parent link="camera"/>
+    <child link="camera_link_optical"/>
+  </joint>
+  <link name="camera_link_optical">
+    <visual>
+      <origin xyz="0 0 0" rpy="0 0 0"/>
+      <geometry>
+        <box size="0.05 0.04 0.04"/>
+      </geometry>
+    </visual>
+    <collision>
+      <origin xyz="0 0 0" rpy="0 0 0"/>
+      <geometry>
+        <box size="0.05 0.05 0.05"/>
+      </geometry>
+    </collision>
+    <inertial>
+      <origin xyz="0 0 0" rpy="0 0 0"/>
+      <mass value="0.1"/>
+      <inertia
+        ixx="1e-6" ixy="0" ixz="0" iyy="1e-6" iyz="0" izz="1e-6"
+      />
+    </inertial>
+  </link>
   <link name="hokuyo">
     <visual>
